File: unsurv_offline_pcb/main/unsurv_offline_pcb.kicad_pcb (KiCad board)
At the start: 4 copper layers, 35 x 50 mm, 62 parts, among them J1 USB_B_Micro, J2 S2B-PH-SM4-TB_LF__SN_, J3 1.27mm_female_connector, Q1 Q_PMOS_GSD, Q2 UMH3N, SW1 SW_DIP_x01, U1 MCP73831-2-OT, U2 APX803L20, U3 AP2112K-3.3, U4 MPU-6050_NRND, U5 ESP32-WROOM-32, U6 CAM-M8C-0-10, U7 CH340G, U8 RF430CL330H

Commit message: finalized smaller pcb
Parts:
- removed R9: 100k, Resistor_SMD:R_0603_1608Metric
- removed U2: APX803L20, digikey-footprints:SOT-23-3
Connections:
- J2 pad 1: +BATT -> GND
- J2 pad 2: GND -> +BATT
Routing:
- net +BATT: track 21.2 -> 23.1 mm
- net GND: track 101.1 -> 100.3 mm, vias 70 -> 71
Changed lines of the file:
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@@
     (thickness 1.6)
     (drawings 4)
-    (tracks 768)
+    (tracks 769)
     (zones 0)
-    (modules 62)
+    (modules 60)
     (nets 95)
   )
@@
   )
   (setup
-    (last_trace_width 0.25)
+    (last_trace_width 0.35)
     (user_trace_width 0.35)
     (user_trace_width 0.5)
@@
     (fp_line (start -3.95 7.25) (end 3.95 7.25) (layer B.Fab) (width 0.1))
     (pad 1 smd rect (at -1 0 270) (size 1 3.5) (layers B.Cu B.Paste B.Mask)
+      (net 1 GND))
+    (pad 2 smd rect (at 1 0 270) (size 1 3.5) (layers B.Cu B.Paste B.Mask)
       (net 3 +BATT))
-    (pad 2 smd rect (at 1 0 270) (size 1 3.5) (layers B.Cu B.Paste B.Mask)
-      (net 1 GND))
     (pad "" smd rect (at -3.35 5.55 270) (size 1.5 3.4) (layers B.Cu B.Paste B.Mask))
     (pad "" smd rect (at 3.35 5.55 270) (size 1.5 3.4) (layers B.Cu B.Paste B.Mask))
@@
   )
   (module Resistor_SMD:R_0603_1608Metric (layer B.Cu)
-    (at 81.25 109.5 90)
-    (descr "Resistor SMD 0603 (1608 Metric), square (rectangular) end terminal, IPC_7351 nominal, (Body size source: http://www.tortai-tech.com/upload/download/2011102023233369053.pdf), generated with kicad-footprint-generator")
-    (tags resistor)
-    (attr smd)
-    (fp_text reference R9 (at 2.1 -0.05 180) (layer B.SilkS)
-      (effects (font (size 0.8 0.8) (thickness 0.1)) (justify mirror))
-    )
-    (fp_text value 100k (at 0 -1.43 90) (layer B.Fab)
-      (effects (font (size 1 1) (thickness 0.15)) (justify mirror))
-    )
-    (fp_line (start -0.8 -0.4) (end -0.8 0.4) (layer B.Fab) (width 0.1))
-    (fp_line (start -0.8 0.4) (end 0.8 0.4) (layer B.Fab) (width 0.1))
-    (fp_line (start 0.8 0.4) (end 0.8 -0.4) (layer B.Fab) (width 0.1))
-    (fp_line (start 0.8 -0.4) (end -0.8 -0.4) (layer B.Fab) (width 0.1))
-    (fp_line (start -0.162779 0.51) (end 0.162779 0.51) (layer B.SilkS) (width 0.12))
-    (fp_line (start -0.162779 -0.51) (end 0.162779 -0.51) (layer B.SilkS) (width 0.12))
-    (fp_line (start -1.48 -0.73) (end -1.48 0.73) (layer B.CrtYd) (width 0.05))
-    (fp_line (start -1.48 0.73) (end 1.48 0.73) (layer B.CrtYd) (width 0.05))
-    (fp_line (start 1.48 0.73) (end 1.48 -0.73) (layer B.CrtYd) (width 0.05))
-    (fp_line (start 1.48 -0.73) (end -1.48 -0.73) (layer B.CrtYd) (width 0.05))
-    (fp_text user %R (at 0 0 90) (layer B.Fab)
-      (effects (font (size 1 1) (thickness 0.15)) (justify mirror))
-    )
-    (pad 1 smd roundrect (at -0.7875 0 90) (size 0.875 0.95) (layers B.Cu B.Paste B.Mask) (roundrect_rratio 0.25)
-      (net 24 BATTALARM))
-    (pad 2 smd roundrect (at 0.7875 0 90) (size 0.875 0.95) (layers B.Cu B.Paste B.Mask) (roundrect_rratio 0.25)
-      (net 4 +3V3))
-    (model ${KISYS3DMOD}/Resistor_SMD.3dshapes/R_0603_1608Metric.wrl
-      (at (xyz 0 0 0))
-      (scale (xyz 1 1 1))
-      (rotate (xyz 0 0 0))
-    )
-  )
-  (module Resistor_SMD:R_0603_1608Metric (layer B.Cu)
     (at 98.9875 114.6)
     (descr "Resistor SMD 0603 (1608 Metric), square (rectangular) end terminal, IPC_7351 nominal, (Body size source: http://www.tortai-tech.com/upload/download/2011102023233369053.pdf), generated with kicad-footprint-generator")
@@
       (rotate (xyz 0 0 0))
     )
-  )
-  (module digikey-footprints:SOT-23-3 (layer B.Cu)
-    (at 78.25 110 270)
-    (attr smd)
-    (fp_text reference U2 (at -2.6 1.25) (layer B.SilkS)
-      (effects (font (size 0.8 0.8) (thickness 0.1)) (justify mirror))
-    )
-    (fp_text value APX803L20 (at 0.025 -3.25 90) (layer B.Fab)
-      (effects (font (size 1 1) (thickness 0.15)) (justify mirror))
-    )
-    (fp_line (start -1.825 1.95) (end 1.825 1.95) (layer B.CrtYd) (width 0.05))
-    (fp_line (start -1.825 1.95) (end -1.825 -1.95) (layer B.CrtYd) (width 0.05))
-    (fp_line (start 1.825 -1.95) (end -1.825 -1.95) (layer B.CrtYd) (width 0.05))
-    (fp_line (start 1.825 1.95) (end 1.825 -1.95) (layer B.CrtYd) (width 0.05))
-    (fp_line (start -0.175 1.65) (end -0.45 1.65) (layer B.SilkS) (width 0.1))
-    (fp_line (start -0.45 1.65) (end -0.825 1.375) (layer B.SilkS) (width 0.1))
-    (fp_line (start -0.825 1.375) (end -0.825 1.325) (layer B.SilkS) (width 0.1))
-    (fp_line (start -0.825 1.325) (end -1.6 1.325) (layer B.SilkS) (width 0.1))
-    (fp_line (start -0.7 1.325) (end -0.7 -1.525) (layer B.Fab) (width 0.1))
-    (fp_line (start -0.425 1.525) (end 0.7 1.525) (layer B.Fab) (width 0.1))
-    (fp_line (start -0.425 1.525) (end -0.7 1.325) (layer B.Fab) (width 0.1))
-    (fp_line (start -0.35 -1.65) (end -0.825 -1.65) (layer B.SilkS) (width 0.1))
-    (fp_line (start -0.825 -1.65) (end -0.825 -1.3) (layer B.SilkS) (width 0.1))
-    (fp_line (start 0.825 -1.425) (end 0.825 -1.3) (layer B.SilkS) (width 0.1))
-    (fp_line (start 0.825 -1.35) (end 0.825 -1.65) (layer B.SilkS) (width 0.1))
-    (fp_line (start 0.825 -1.65) (end 0.375 -1.65) (layer B.SilkS) (width 0.1))
-    (fp_line (start 0.45 1.65) (end 0.825 1.65) (layer B.SilkS) (width 0.1))
-    (fp_line (start 0.825 1.65) (end 0.825 1.35) (layer B.SilkS) (width 0.1))
-    (fp_text user %R (at -0.125 -0.15 90) (layer B.Fab)
-      (effects (font (size 1 1) (thickness 0.15)) (justify mirror))
-    )
-    (fp_line (start -0.7 -1.52) (end 0.7 -1.52) (layer B.Fab) (width 0.1))
-    (fp_line (start 0.7 -1.52) (end 0.7 1.52) (layer B.Fab) (width 0.1))
-    (pad 3 smd rect (at 1.05 0 270) (size 1.3 0.6) (layers B.Cu B.Paste B.Mask)
-      (net 3 +BATT) (solder_mask_margin 0.07))
-    (pad 2 smd rect (at -1.05 -0.95 270) (size 1.3 0.6) (layers B.Cu B.Paste B.Mask)
-      (net 24 BATTALARM) (solder_mask_margin 0.07))
-    (pad 1 smd rect (at -1.05 0.95 270) (size 1.3 0.6) (layers B.Cu B.Paste B.Mask)
-      (net 1 GND) (solder_mask_margin 0.07))
   )
   (module digikey-footprints:QFN-24-1EP_4x4mm (layer B.Cu)
@@
   (segment (start 101.755 97.345) (end 100.1 99) (width 0.25) (layer B.Cu) (net 1))
   (via (at 81.5 121.3) (size 0.6) (drill 0.3) (layers F.Cu B.Cu) (net 1))
-  (segment (start 84.15 120.85) (end 81.95 120.85) (width 0.25) (layer B.Cu) (net 1))
-  (segment (start 81.95 120.85) (end 81.5 121.3) (width 0.25) (layer B.Cu) (net 1))
   (segment (start 97.675001 114.900001) (end 97.675001 115.594999) (width 0.25) (layer F.Cu) (net 1))
   (segment (start 97.2 113.9875) (end 97.2 114.425) (width 0.25) (layer F.Cu) (net 1))
@@
   (segment (start 100.947634 121.427634) (end 99.386634 121.427634) (width 0.25) (layer B.Cu) (net 1))
   (segment (start 102 122.48) (end 100.947634 121.427634) (width 0.25) (layer B.Cu) (net 1))
+  (via (at 85.7 117.6) (size 0.6) (drill 0.3) (layers F.Cu B.Cu) (net 1))
+  (segment (start 84.15 118.85) (end 84.45 118.85) (width 0.35) (layer B.Cu) (net 1))
+  (segment (start 84.45 118.85) (end 85.7 117.6) (width 0.35) (layer B.Cu) (net 1))
   (via (at 90.100006 118.3) (size 0.8) (drill 0.4) (layers F.Cu B.Cu) (net 2))
   (segment (start 91.175 119.374994) (end 91.175 120.235) (width 0.35) (layer F.Cu) (net 2))
@@
   (segment (start 77.0625 114.4625) (end 77.28 114.68) (width 0.35) (layer F.Cu) (net 3))
   (segment (start 77.0625 113.5) (end 77.0625 114.4625) (width 0.35) (layer F.Cu) (net 3))
-  (segment (start 82.9 118.85) (end 84.15 118.85) (width 0.35) (layer B.Cu) (net 3))
-  (segment (start 82.05 118) (end 82.9 118.85) (width 0.35) (layer B.Cu) (net 3))
-  (segment (start 82.05 116.75) (end 82.05 118) (width 0.35) (layer B.Cu) (net 3))
-  (segment (start 80.724999 115.424999) (end 82.05 116.75) (width 0.35) (layer B.Cu) (net 3))
   (segment (start 78.024999 115.424999) (end 80.724999 115.424999) (width 0.35) (layer B.Cu) (net 3))
   (segment (start 77.28 114.68) (end 78.024999 115.424999) (width 0.35) (layer B.Cu) (net 3))
@@
   (segment (start 82.6 121.1) (end 82.6 120.619998) (width 0.35) (layer F.Cu) (net 3))
   (segment (start 82.6 120.619998) (end 83.32 119.899998) (width 0.35) (layer F.Cu) (net 3))
-  (segment (start 83.32 119.68) (end 84.15 118.85) (width 0.35) (layer B.Cu) (net 3))
-  (segment (start 83.32 119.899998) (end 83.32 119.68) (width 0.35) (layer B.Cu) (net 3))
+  (segment (start 84.15 120.729998) (end 83.32 119.899998) (width 0.35) (layer B.Cu) (net 3))
+  (segment (start 84.15 120.85) (end 84.15 120.729998) (width 0.35) (layer B.Cu) (net 3))
+  (segment (start 82.9 120.85) (end 81.3 119.25) (width 0.35) (layer B.Cu) (net 3))
+  (segment (start 84.15 120.85) (end 82.9 120.85) (width 0.35) (layer B.Cu) (net 3))
+  (segment (start 81.3 116) (end 80.724999 115.424999) (width 0.35) (layer B.Cu) (net 3))
+  (segment (start 81.3 119.25) (end 81.3 116) (width 0.35) (layer B.Cu) (net 3))
   (via (at 79.4 102) (size 0.8) (drill 0.4) (layers F.Cu B.Cu) (net 4))
   (segment (start 98.2 116.1875) (end 98.2125 116.2) (width 0.25) (layer B.Cu) (net 4))
