File: unsurv_offline_pcb/main/d4_small_pcb.kicad_pcb (KiCad board)
At the start: 4 copper layers, 32 x 45 mm, 54 parts, among them J1 U_FL-R-SMT-1_10_, J2 S2B-PH-SM4-TB_LF__SN_, Q1 UMH3N, Q2 Q_PMOS_GSD, U1 TTGO-Micro32-ESP32, U2 MCP73831-2-OT, U3 CAM-M8C-0-10, U4 AP2112K-3.3, U5 CH340G, U6 RF430CL330H, U7 BMA400-I2C, U8 RFM95W-868S2

Commit message: PCB redesign
Parts:
- removed D4: D_Schottky, Diode_SMD:D_SOD-323
- removed Q2: Q_PMOS_GSD, Package_TO_SOT_SMD:SOT-23
- removed R11: 100k, Resistor_SMD:R_0603_1608Metric
- removed U2: MCP73831-2-OT, Package_TO_SOT_SMD:SOT-23-5
- added C15: 1yF, Capacitor_SMD:C_0603_1608Metric, F.Cu at (24.5, 60.0)
- added U9: PQ2581DLHT, unsurv_offline_pcb_footprints:BQ2581DLHT, F.Cu at (25.3, 58.0)
- C1: value 4.7yF -> 10yF
- C2: value 4.7yF -> 1yF
- R2: value 10k -> 1k
- R3: value 1k -> 10k
- moved R10 46.8 mm to (21.9, 61.8), turned to -90 degrees
- moved C8 46.4 mm to (20.3, 61.8), turned to 90 degrees
- moved U4 42.1 mm to (21.0, 58.2), turned to 90 degrees
- moved C1 39.7 mm to (25.2, 62.4), turned to -90 degrees
- moved C6 39.4 mm to (19.4, 54.4)
- moved C7 35.9 mm to (21.1, 54.4), turned to -90 degrees
- moved D3 35.2 mm to (27.6, 63.6), turned to 180 degrees
- moved R3 33.2 mm to (23.9, 54.4), turned to 90 degrees
- moved CARD1 31.7 mm to (42.7, 29.4), turned to 90 degrees
- moved C2 30.6 mm to (26.9, 60.9), turned to 90 degrees
- moved R2 29.3 mm to (28.6, 60.9), turned to -90 degrees
- moved R16 27.8 mm to (44.3, 48.7), turned to 0 degrees
- moved USB1 23.5 mm to (34.0, 62.0), turned to 0 degrees
- moved R13 23.4 mm to (47.1, 38.7)
- moved C13 22.7 mm to (23.6, 48.5), turned to -90 degrees
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Connections:
- C1 pad 1: GND -> VCC
- C1 pad 2: +BATT -> GND
- C2 pad 2: +5V -> +BATT
- C8 pad 2: Net-(C8-Pad2) -> VCC
- R10 pad 2: Net-(C8-Pad2) -> VCC
- R2 pad 2: GND -> Net-(D3-Pad1)
- R3 pad 2: Net-(D3-Pad1) -> GND
- U1 pad 4: unconnected-(U1-Pad4) -> 36
- U4 pad 1: Net-(C8-Pad2) -> VCC
Routing:
- net GND: track 77.2 -> 10.1 mm, vias 68 -> 67
- net 32: track 62.0 -> 19.0 mm, vias 3 -> 1
- net 23: track 67.2 -> 24.2 mm, vias 3 -> 2
- net +BATT: track 46.4 -> 6.27 mm
- net SCL: track 50.0 -> 82.3 mm, vias 5 -> 6
- net 36: track 0.00 -> 29.8 mm, vias 0 -> 2
- net SDA: track 46.1 -> 71.2 mm, vias 4 -> 6
- net 19: track 41.3 -> 18.8 mm, vias 1 -> 3
- net 18: track 43.8 -> 21.6 mm, vias 1 -> 3
- net 34: track 51.2 -> 30.6 mm
- net 14: track 43.1 -> 25.5 mm
- net Net-(C8-Pad2): track 12.7 -> 0.00 mm
- net 33: track 51.0 -> 39.1 mm, vias 4 -> 2
- net VCC: track 0.00 -> 11.1 mm
- net 35: track 25.6 -> 16.2 mm
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- added copper zone on In1.Cu, net +3V3
- added copper zone on In1.Cu, net +5V
- removed copper zone on In1.Cu, net GND
