File: unsurv_offline_pcb/main/d4_small_pcb.kicad_pcb (KiCad board)
At the start: 4 copper layers, 32 x 45 mm, 59 parts, among them J1 S2B-PH-SM4-TB_LF__SN_, J2 U_FL-R-SMT-1_10_, Q1 UMH3N, U1 BQ25180, U2 TTGO-Micro32-ESP32, U3 CAM-M8C, U4 RFM95W-868S2, U5 AP2112K-3.3, U6 CH340G, U7 RF430CL330HIRGTR‎, U8 BMA400

Commit message: certification test
Parts:
- D1_or1: value LED -> LED1
- D2_g1: value LED -> LED2
Changed lines of the file:
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@@
       (effects (font (size 0.5 0.5) (thickness 0.1)))
     )
-    (fp_text value "LED" (at 0 1.77 unlocked) (layer "F.Fab")
+    (fp_text value "LED1" (at 0 1.77 unlocked) (layer "F.Fab")
       (effects (font (size 1 1) (thickness 0.15)))
     )
@@
       (effects (font (size 0.5 0.5) (thickness 0.1)))
     )
-    (fp_text value "LED" (at 0 1.77 unlocked) (layer "F.Fab")
+    (fp_text value "LED2" (at 0 1.77 unlocked) (layer "F.Fab")
       (effects (font (size 1 1) (thickness 0.15)))
     )

Commit message: new footprints
Parts:
- added C5: 10µF, Capacitor_SMD:C_0603_1608Metric, F.Cu at (23.5, 52.8)
- added L1: L_Ferrite, Inductor_SMD:L_0603_1608Metric, F.Cu at (28.6, 60.5)
- added L2: L_Ferrite, Inductor_SMD:L_0603_1608Metric, F.Cu at (25.1, 52.8)
- moved C16 0.83 mm to (24.3, 50.5)
- moved R7 0.83 mm to (24.3, 47.2)
- moved R6 0.82 mm to (24.3, 48.9)
- moved TP7 0.75 mm to (27.1, 54.1)
- moved TP8 0.75 mm to (29.7, 54.1)
- renumbered C9 to C10, C10 to C11, C11 to C12, C12 to C13, C13 to C14, C14 to C15, C15 to C16, C5 to C6, C6 to C7, C7 to C8, C8 to C9
Routing:
- net +3V3: track 57.1 -> 62.2 mm, vias 19 -> 18
- net +5V: track 6.06 -> 7.78 mm
- net GND: vias 76 -> 75
