File: hardware/main/d4_small_pcb.kicad_sch (KiCad schematic)
At the start: 62 parts, among them J1 S2B-PH-SM4-TB_LF__SN_, J2 U_FL-R-SMT-1_10_, Q1 UMH3N, U1 BQ25180, U2 TTGO-Micro32-ESP32, U3 CAM-M8C, U4 RFM95W-868S2, U5 AP2112K-3.3, U6 CH340G, U7 RF430CL330HIRGTR‎, U8 BMA400

Commit message: update BMA400 +BQ25180 footprints
Parts:
- U8: footprint unsurv_offline_pcb_footprints:BMA400_regular -> unsurv:BMA400_regular

Commit message: repair project + update 3D model path for KiCad 8
Parts:
- U1: footprint unsurv:BQ25180 -> unsurv_offline_pcb_footprints:BQ25180
- U8: footprint unsurv:BMA400_regular -> unsurv_offline_pcb_footprints:BMA400_regular
